Commit message: add pen model

File: crane_x7_description/urdf/pen.urdf (robot description, URDF)
Before this commit: robot pen, 1 links, 1 joints
Joints:
- joint pen_joint: origin xyz=0 0 0.05 rpy=0 1.570796326795 0 -> xyz=0 0 0.1 rpy=0 1.570796326795 0

Commit message: add new hude

File: crane_x7_description/urdf/pen.urdf (robot description, URDF)
Before this commit: robot pen, 1 links, 1 joints
Links:
- link pen_link: geometry visual mesh filename=package://crane_x7_description/meshes/pencase/coordinate.dae
Joints:
- joint pen_joint: origin xyz=0 0 0.1 rpy=0 1.570796326795 0 -> xyz=0 0.14 0.083 rpy=0 0 -1.570796
