Commit message: bag fix

File: crane_x7_description/urdf/crane_x7.xacro (robot description, xacro)
@@ -1,3 +1,6 @@
 <?xml version="1.0"?>
+<!-- これがコメントアウトのやり方です   -->
+<!--これを用いて、筆の表示を消したい場合は,<xacro:include filename="$(find crane_x7_description)/urdf/pen.urdf"/>を上記の方法で
+	コメントアウトしていただくと消えます-->
 <robot xmlns:xacro="http://ros.org/wiki/xacro">
   <xacro:include filename="$(find crane_x7_description)/urdf/crane_x7_mounting_plate.xacro"/>

File: crane_x7_description/urdf/pen.urdf (robot description, URDF)
Before this commit: robot pen, 1 links, 1 joints
Links:
- link pen_link: geometry visual mesh filename=package://crane_x7_description/meshes/pencase/fix.dae
Joints:
- joint pen_joint: origin xyz=0 0.14 0.083 rpy=0 0 -1.570796 -> xyz=0 -0.027 0.083 rpy=0 0 -1.570796
